File: redux/zoom.kicad_sch (KiCad schematic)
At the start: 161 parts, among them U10 1NB4-5040, U11 1NB4-5040, U12 1NB4-5040, U14 1821-4731, U2 LM2991, U7 LT1086-CM, U77 74LVC08, U78 74LVC08, U8 1NB4-5040, U9 1NB4-5040

Commit message: redux work
Parts:
- removed RP1, RP2: 150, fp:SOIC-16W_5.3x10.2mm_P1.27mm, symbol 16717a:RPack8
- removed RP14, RP15: 330, fp:SOIC-16W_5.3x10.2mm_P1.27mm, symbol 16717a:RPack8
- added C1: 3.3n, fp:C0603, symbol Device:C_Small
- added R1, R2, R7, R8: 330, fp:R_Array_Convex_4x0603, symbol Device:R_Pack04
- added R3, R4, R5, R6: 150, fp:R_Array_Convex_4x0603, symbol Device:R_Pack04
Connections:
- net +3.3V: now also R1.5 (R4.2), R1.6 (R3.2), R1.7 (R2.2), R1.8 (R1.2), R2.5 (R4.2), R2.6 (R3.2), R2.7 (R2.2), R2.8 (R1.2), R7.5 (R4.2), R7.6 (R3.2), R7.7 (R2.2), R7.8 (R1.2), R8.5 (R4.2), R8.6 (R3.2), R8.7 (R2.2), R8.8 (R1.2)
- net -1.7V: now also C1.2
- net GND: now also C1.1, R5.5 (R4.2), R5.6 (R3.2)
- net ZCCTRL0: now also R6.8 (R1.2)
- net ZCCTRL1: now also R6.5 (R4.2)
- net ZCCTRL2: now also R6.6 (R3.2)
- net ZCCTRL3: now also R6.7 (R2.2)
- net ZCCTRL5: now also R5.7 (R2.2)
- net ZCCTRL6: now also R5.8 (R1.2)
- net ZD_{0}: now also R4.1 (R1.1)
- net ZD_{1}: now also R4.2 (R2.1)
- net ZD_{2}: now also R4.3 (R3.1)
- net ZD_{3}: now also R4.4 (R4.1)
- net ZD_{4}: now also R3.1 (R1.1)
- net ZD_{5}: now also R3.2 (R2.1)
- net ZD_{6}: now also R3.3 (R3.1)
- net ZD_{7}: now also R3.4 (R4.1)
- net at U14.5 (CTRL3): now also R6.2 (R2.1), R8.3 (R3.1)
- net at U14.4 (CTRL2): now also R6.3 (R3.1), R8.2 (R2.1)
- net at U14.22 (CTRL6): now also R5.1 (R1.1), R7.4 (R4.1)
- net at U14.21 (CTRL5): now also R5.2 (R2.1), R7.3 (R3.1)
- net at U14.20 (CTRL4): now also R5.3 (R3.1), R7.2 (R2.1)
- net at U14.94 (CTRL1): now also R6.4 (R4.1), R8.1 (R1.1)
- net at U14.6 (CTRL0): now also R6.1 (R1.1), R8.4 (R4.1)
- net at U14.17 (D_{0}): now also R2.1 (R1.1), R4.8 (R1.2)
- net at U14.16 (D_{1}): now also R2.2 (R2.1), R4.7 (R2.2)
- net at U14.15 (D_{2}): now also R2.3 (R3.1), R4.6 (R3.2)
- net at U14.14 (D_{3}): now also R2.4 (R4.1), R4.5 (R4.2)
- net at U14.12 (D_{4}): now also R1.1 (R1.1), R3.8 (R1.2)
- net at U14.11 (D_{5}): now also R1.2 (R2.1), R3.7 (R2.2)
- net at U14.10 (D_{6}): now also R1.3 (R3.1), R3.6 (R3.2)
- net at U14.9 (D_{7}): now also R1.4 (R4.1), R3.5 (R4.2)

Commit message: Rework acquisition ASIC routing
Parts:
- added C10, C9: 51n, fp:C0805, symbol Device:C_Small
Connections:
- net +3.3V: now also U2.2 (~{ON}/OFF), C10.1, C9.1
- net +3.3VP: no longer U2.2 (~{ON}/OFF)
- net GND: now also C10.2, C9.2
- net ZD_{1}: no longer U12.40 (NC)
- net ZD_{2}: no longer U12.38 (NC)
- net ZD_{3}: no longer U12.37 (NC)
- no-connect marks 31 -> 34
