File: redux/probe_cable.kicad_sch (KiCad schematic)
At the start: 1 part, among them J1 Conn_02x30_Odd_Even

Commit message: Fix SY89421V pin 9 held low instead of floating
Parts:
- J1: footprint fp:Probe_Connector -> fp:Probe_Connector_MountingHoles
Changed lines of the file:
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@@
 			)
 		)
-		(property "Footprint" "fp:Probe_Connector"
+		(property "Footprint" "fp:Probe_Connector_MountingHoles"
 			(at 119.38 80.01 0)
 			(effects
