File: redux/acquisition.kicad_sch (KiCad schematic)
At the start: 17 parts, among them U21 1821-3936

Commit message: Rework acquisition ASIC routing
Parts:
- U21: footprint fp:BGA-479_40.5mm_P1.27mm -> fp:BGA-479_40.5mm_P1.27mm_VIP
Changed lines of the file:
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@@
 			)
 		)
-		(property "Footprint" "fp:BGA-479_40.5mm_P1.27mm"
+		(property "Footprint" "fp:BGA-479_40.5mm_P1.27mm_VIP"
 			(at 292.1 304.8 0)
 			(effects

Commit message: rev 1 (submitted to jlc)
Parts:
- added TP11, TP13, TP15, TP17, TP19, TP2, TP21, TP23, TP25, TP27, TP29, TP31, TP33, TP4, TP5, TP7, TP9: TestPoint_Small, fp:TestPoint, symbol 16717a:TestPoint_Small
Connections:
- net SC_{8}: now also TP2.1
- net SD_{128}: now also TP33.1
- net SD_{129}: now also TP31.1
- net SD_{130}: now also TP29.1
- net SD_{131}: now also TP27.1
- net SD_{132}: now also TP25.1
- net SD_{133}: now also TP23.1
- net SD_{134}: now also TP21.1
- net SD_{135}: now also TP19.1
- net SD_{136}: now also TP17.1
- net SD_{137}: now also TP15.1
- net SD_{138}: now also TP13.1
- net SD_{139}: now also TP11.1
- net SD_{140}: now also TP9.1
- net SD_{141}: now also TP7.1
- net SD_{142}: now also TP5.1
- net SD_{143}: now also TP4.1
