File: original/acquisition.kicad_sch (KiCad schematic)
At the start: 17 parts, among them U21 1821-3936

Commit message: clean up routing & add test points on original design
Parts:
- added TP145, TP146, TP147, TP148, TP149, TP150, TP151, TP152, TP153, TP154, TP155, TP156, TP157, TP158, TP159, TP160, TP177, TP178, TP179, TP180, TP181, TP182, TP183, TP184, TP185, TP186, TP187, TP188, TP189, TP190, TP191, TP192, TP209, TP210, TP211, TP212, TP213, TP214, TP215, TP216, TP217, TP218, TP219, TP220, TP221, TP222, TP223, TP224, TP241, TP242, TP243, TP244, TP245, TP246, TP247, TP248, TP249, TP250, TP251, TP252, TP253, TP254, TP255, TP256, TP273, TP274, TP275, TP276, TP277, TP278, TP279, TP280, TP281, TP282, TP283, TP284, TP285, TP286, TP287, TP288, TP305, TP306, TP307, TP308, TP309, TP310, TP311, TP312, TP313, TP314, TP315, TP316, TP317, TP318, TP319, TP320, TP337, TP338, TP339, TP340, TP341, TP342, TP343, TP344, TP345, TP346, TP347, TP348, TP349, TP350, TP351, TP352, TP369, TP372, TP374, TP376, TP377, TP378, TP379, TP380, TP381, TP382, TP383, TP384, TP401, TP402, TP403, TP404, TP405, TP406, TP407, TP408, TP409, TP410, TP411, TP412, TP413, TP414, TP415, TP416, TP425, TP426, TP427, TP428, TP429, TP430, TP431, TP432, TP434, TP451, TP452, TP453, TP454, TP455, TP456, TP457, TP458, TP459, TP460, TP461, TP462, TP463, TP464, TP465, TP466, TP483, TP484, TP485, TP486, TP487, TP488, TP489, TP490, TP491, TP492, TP493, TP494, TP495, TP496, TP497, TP498, TP501, TP502, TP505, TP506, TP556, TP558, TP560, TP562, TP615, TP617, TP642, TP644, TP646, TP648, TP877: ~, fp:TestPoint, symbol 16717a:TestPoint_Small
Connections:
- net +3.3V: now also TP560.1, TP617.1, TP644.1
- net GND: now also TP562.1, TP615.1, TP642.1
- net PA_{0}: now also TP483.1
- net PA_{10}: now also TP493.1
- net PA_{11}: now also TP494.1
- net PA_{12}: now also TP495.1
- net PA_{13}: now also TP496.1
- net PA_{14}: now also TP497.1
- net PA_{15}: now also TP498.1
- net PA_{1}: now also TP484.1
- net PA_{2}: now also TP485.1
- net PA_{3}: now also TP486.1
- net PA_{4}: now also TP487.1
- net PA_{5}: now also TP488.1
- net PA_{6}: now also TP489.1
- net PA_{7}: now also TP490.1
- net PA_{8}: now also TP491.1
- net PA_{9}: now also TP492.1
- net PA_{CLK}: now also TP501.1
- net PB_{0}: now also TP451.1
- net PB_{10}: now also TP461.1
- net PB_{11}: now also TP462.1
- net PB_{12}: now also TP463.1
- net PB_{13}: now also TP464.1
- net PB_{14}: now also TP465.1
- net PB_{15}: now also TP466.1
- net PB_{1}: now also TP452.1
- net PB_{2}: now also TP453.1
- net PB_{3}: now also TP454.1
- net PB_{4}: now also TP455.1
- net PB_{5}: now also TP456.1
- net PB_{6}: now also TP457.1
- net PB_{7}: now also TP458.1
- net PB_{8}: now also TP459.1
- net PB_{9}: now also TP460.1
- net PB_{CLK}: now also TP505.1
- net SC_{0}: now also TP434.1
- net SC_{1}: now also TP425.1
- net SC_{2}: now also TP426.1
- net SC_{3}: now also TP427.1
- net SC_{4}: now also TP428.1
- net SC_{5}: now also TP429.1
- net SC_{6}: now also TP430.1
- net SC_{7}: now also TP431.1
- net SC_{8}: now also TP432.1
- net SD_{0}: now also TP401.1
- net SD_{100}: now also TP309.1
- net SD_{101}: now also TP310.1
- net SD_{102}: now also TP311.1
- net SD_{103}: now also TP312.1
- net SD_{104}: now also TP313.1
- net SD_{105}: now also TP314.1
- net SD_{106}: now also TP315.1
- net SD_{107}: now also TP316.1
- net SD_{108}: now also TP317.1
- net SD_{109}: now also TP318.1
- net SD_{10}: now also TP411.1
- net SD_{110}: now also TP319.1
- net SD_{111}: now also TP320.1
- net SD_{112}: now also TP337.1
- net SD_{113}: now also TP338.1
- net SD_{114}: now also TP339.1
- net SD_{115}: now also TP340.1
- net SD_{116}: now also TP341.1
- net SD_{117}: now also TP342.1
- net SD_{118}: now also TP343.1
- net SD_{119}: now also TP344.1
- net SD_{11}: now also TP412.1
- net SD_{120}: now also TP345.1
- net SD_{121}: now also TP346.1
- net SD_{122}: now also TP347.1
- net SD_{123}: now also TP348.1
- net SD_{124}: now also TP349.1
- net SD_{125}: now also TP350.1
- net SD_{126}: now also TP351.1
- net SD_{127}: now also TP352.1
- net SD_{128}: now also TP369.1
- net SD_{12}: now also TP413.1
- net SD_{131}: now also TP372.1
- net SD_{133}: now also TP374.1
- net SD_{135}: now also TP376.1
- net SD_{136}: now also TP377.1
- net SD_{137}: now also TP378.1
- net SD_{138}: now also TP379.1
- net SD_{139}: now also TP380.1
- net SD_{13}: now also TP414.1
- net SD_{140}: now also TP381.1
- net SD_{141}: now also TP382.1
- net SD_{142}: now also TP383.1
- net SD_{143}: now also TP384.1
- net SD_{14}: now also TP415.1
- net SD_{15}: now also TP416.1
- net SD_{16}: now also TP145.1
- net SD_{17}: now also TP146.1
- net SD_{18}: now also TP147.1
- net SD_{19}: now also TP148.1
- net SD_{1}: now also TP402.1
- net SD_{20}: now also TP149.1
- net SD_{21}: now also TP150.1
- net SD_{22}: now also TP151.1
- net SD_{23}: now also TP152.1
- net SD_{24}: now also TP153.1
- net SD_{25}: now also TP154.1
- net SD_{26}: now also TP155.1
- net SD_{27}: now also TP156.1
- net SD_{28}: now also TP157.1
- net SD_{29}: now also TP158.1
- net SD_{2}: now also TP403.1
- net SD_{30}: now also TP159.1
- net SD_{31}: now also TP160.1
- net SD_{32}: now also TP177.1
- net SD_{33}: now also TP178.1
- net SD_{34}: now also TP179.1
- net SD_{35}: now also TP180.1
- net SD_{36}: now also TP181.1
- net SD_{37}: now also TP182.1
- net SD_{38}: now also TP183.1
- net SD_{39}: now also TP184.1
- net SD_{3}: now also TP404.1
- net SD_{40}: now also TP185.1
- net SD_{41}: now also TP186.1
- net SD_{42}: now also TP187.1
- net SD_{43}: now also TP188.1
- net SD_{44}: now also TP189.1
- net SD_{45}: now also TP190.1
- net SD_{46}: now also TP191.1
- net SD_{47}: now also TP192.1
- net SD_{48}: now also TP209.1
- net SD_{49}: now also TP210.1
- net SD_{4}: now also TP405.1
- net SD_{50}: now also TP211.1
- net SD_{51}: now also TP212.1
- net SD_{52}: now also TP213.1
- net SD_{53}: now also TP214.1
- net SD_{54}: now also TP215.1
- net SD_{55}: now also TP216.1
- net SD_{56}: now also TP217.1
- net SD_{57}: now also TP218.1
- net SD_{58}: now also TP219.1
- net SD_{59}: now also TP220.1
- net SD_{5}: now also TP406.1
- net SD_{60}: now also TP221.1
- net SD_{61}: now also TP222.1
- net SD_{62}: now also TP223.1
- net SD_{63}: now also TP224.1
- net SD_{64}: now also TP241.1
- net SD_{65}: now also TP242.1
- net SD_{66}: now also TP243.1
- net SD_{67}: now also TP244.1
- net SD_{68}: now also TP245.1
- net SD_{69}: now also TP246.1
- net SD_{6}: now also TP407.1
- net SD_{70}: now also TP247.1
- net SD_{71}: now also TP248.1
- net SD_{72}: now also TP249.1
- net SD_{73}: now also TP250.1
- net SD_{74}: now also TP251.1
- net SD_{75}: now also TP252.1
- net SD_{76}: now also TP253.1
- net SD_{77}: now also TP254.1
- net SD_{78}: now also TP255.1
- net SD_{79}: now also TP256.1
- net SD_{7}: now also TP408.1
- net SD_{80}: now also TP273.1
- net SD_{81}: now also TP274.1
- net SD_{82}: now also TP275.1
- net SD_{83}: now also TP276.1
- net SD_{84}: now also TP277.1
- net SD_{85}: now also TP278.1
- net SD_{86}: now also TP279.1
- net SD_{87}: now also TP280.1
- net SD_{88}: now also TP281.1
- net SD_{89}: now also TP282.1
- net SD_{8}: now also TP409.1
- net SD_{90}: now also TP283.1
- net SD_{91}: now also TP284.1
- net SD_{92}: now also TP285.1
- net SD_{93}: now also TP286.1
- net SD_{94}: now also TP287.1
- net SD_{95}: now also TP288.1
- net SD_{96}: now also TP305.1
- net SD_{97}: now also TP306.1
- net SD_{98}: now also TP307.1
- net SD_{99}: now also TP308.1
- net SD_{9}: now also TP410.1
- net V_{BB}: now also TP877.1
- net ZOOM_TRIG: now also TP648.1
- net ~{PA_{CLK}}: now also TP502.1
- net ~{PB_{CLK}}: now also TP506.1
- net at R1227.1, R1228.1, U21.AA26 (???): now also TP558.1
- net at R1227.2, R1228.2, U21.AB27 (???): now also TP556.1
- net at R1218.1, U21.AA27 (???): now also TP646.1
Other:
- moved on the sheet: R1219
