File: original/board_stacking.kicad_sch (KiCad schematic)
At the start: 52 parts, among them Q1001 MRF9511LT1, Q1003 MRF9511LT1, Q1005 MRF9511LT1, Q1007 MRF9511LT1, Q1009 MRF9511LT1, Q1011 MRF9511LT1, U18 MC100LVEL16, U20 MC100LVEL16, U24 MC100LVEL16

Commit message: clean up routing & add test points on original design
Parts:
- added TP618, TP619, TP620, TP621, TP622, TP623, TP624, TP625, TP626, TP627, TP628, TP631, TP632, TP634, TP636, TP637, TP638, TP639: ~, fp:TestPoint, symbol 16717a:TestPoint_Small
Connections:
- net DOUTA_{1}+: now also TP634.1
- net DOUTA_{2}+: now also TP639.1
- net DOUTA_{2}-: now also TP638.1
- net DOUTB_{0}+: now also TP627.1
- net DOUTB_{0}-: now also TP628.1
- net DOUTB_{1}+: now also TP632.1
- net DOUTB_{1}-: now also TP631.1
- net DOUTB_{2}+: now also TP637.1
- net DOUTB_{2}-: now also TP636.1
- net D_{0}: now also TP619.1
- net D_{1}: now also TP621.1
- net D_{2}: now also TP623.1
- net ~{D_{0}}: now also TP618.1
- net ~{D_{1}}: now also TP620.1
- net ~{D_{2}}: now also TP622.1
- net at Q1001.3 (B), R1159.2: now also TP625.1
- net at Q1011.2 (E), Q1011.4 (E), R1222.1: now also TP624.1
- net at Q1001.2 (E), Q1001.4 (E), R1160.1: now also TP626.1
