File: original/original.kicad_sch (KiCad schematic)
At the start: 244 parts, among them J11 DNP, J12 DNP, J13 DNP, J14 Backplane, J3 Common, J4 Ext-2, J5 Ext-1, J6 Master, J7 Ext+1, J8 Ext+2, M1000 Bracket, Q1 MMBT3906, U1 MC100LVEL16, U13 MC100LVEL14, U15 SY89421V, U16 LM311, U34 AD7841, U44 AD586, U45 AD586, U62 LT1086-ADJ, U63 LT1086-ADJ, U64 16715-89002, U65 74CBT3125, U66 SG-615P 19.6608MHz, U67 SN74FB2040, U68 MC100LVEL11, U73 MC100LVEL16, U74 MC10EL34, U75 PCF8584, U76 74ABT540, U79 NEL HS-2810 101MHz

Commit message: fix original version ECL routing to ASICs
Parts:
- R1106: value 316 -> 215
Connections:
- net +2.5V renamed +2.1V
Changed lines of the file:
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@@
 		)
 	)
-	(text_box "The inverting input voltage divider here is set up to generate around 2.1V, which seems approximately the correct V_{BB} for the zoom clock distribution chip's weird \"5V ECL with V_{EE} at -1.3V\".  This makes me think this whole comparator is just a big, slow level translator for some kind of feedback signal from the zoom chip."
-		(exclude_from_sim no)
-		(at 382.27 74.93 0)
-		(size 40.64 20.32)
-		(stroke
-			(width 0)
-			(type default)
-		)
-		(fill
-			(type none)
-		)
-		(effects
-			(font
-				(size 1.27 1.27)
-			)
-			(justify left top)
-		)
-	)
 	(text_box "The 16500A backplane bus had 8 dedicated bidirectional data lines and separate unidirectional address lines.  The 16700A service manual notes that the 16700 bus is backwards compatible with that, but has been extended to allow a 16b mode with multiplexed data/address.\n\nSince all these signals just go straight into the bus interface FPGA, I don't really know what's what, so I've just named these bus interface (\"BIF\") signals based on their pin number on the backplane.\n\nNote there is also an 8b open collector bus, which I believe is what the service manual refers to as the IMB (inter-module bus) and is used for synchronizing triggers between modules.  I'm calling that bus ~{EVENT_{[0..7]}}"
 		(exclude_from_sim no)
@@
 			)
 		)
-		(property "Value" "316"
+		(property "Value" "215"
 			(at 775.97 113.0299 0)
 			(effects
@@
 	)
 	(symbol
-		(lib_id "16717a:+2.5V")
+		(lib_id "16717a:+2.1V")
 		(at 746.76 148.59 0)
 		(mirror y)
@@
 			)
 		)
-		(property "Value" "+2.5V"
-			(at 746.76 143.51 0)
+		(property "Value" "+2.1V"
+			(at 749.3 147.3199 0)
 			(effects
 				(font
 					(size 1.27 1.27)
 				)
+				(justify right)
 			)
 		)
@@
 			)
 		)
-		(property "Description" "Power symbol creates a global label with name \"+1.5V\""
+		(property "Description" "Power symbol creates a global label with name \"+2.1V\""
 			(at 746.76 148.59 0)
 			(effects
@@
 	)
 	(symbol
-		(lib_id "16717a:+2.5V")
+		(lib_id "16717a:+2.1V")
 		(at 763.27 355.6 0)
 		(unit 1)
@@
 			)
 		)
-		(property "Value" "+2.5V"
-			(at 763.27 350.52 0)
+		(property "Value" "+2.1V"
+			(at 765.81 354.3299 0)
 			(effects
 				(font
 					(size 1.27 1.27)
 				)
+				(justify left)
 			)
 		)
@@
 			)
 		)
-		(property "Description" "Power symbol creates a global label with name \"+1.5V\""
+		(property "Description" "Power symbol creates a global label with name \"+2.1V\""
 			(at 763.27 355.6 0)
 			(effects
@@
 	)
 	(symbol
-		(lib_id "16717a:+2.5V")
+		(lib_id "16717a:+2.1V")
 		(at 817.88 100.33 270)
 		(unit 1)
@@
 			)
 		)
-		(property "Value" "+2.5V"
+		(property "Value" "+2.1V"
 			(at 821.69 100.3299 90)
 			(effects
@@
 			)
 		)
-		(property "Description" "Power symbol creates a global label with name \"+1.5V\""
+		(property "Description" "Power symbol creates a global label with name \"+2.1V\""
 			(at 817.88 100.33 0)
 			(effects

Commit message: clean up routing & add test points on original design
Parts:
- added TP1, TP1000, TP1001, TP1002, TP1003, TP1004, TP1005, TP1006, TP1008, TP1009, TP1010, TP1011, TP1012, TP1013, TP1014, TP1015, TP1016, TP1017, TP1018, TP1019, TP1020, TP1021, TP1022, TP1023, TP1024, TP1025, TP1026, TP1027, TP1028, TP1029, TP1030, TP1031, TP1032, TP1033, TP1034, TP1035, TP1036, TP1037, TP1038, TP1039, TP1040, TP1041, TP1042, TP1043, TP1044, TP1045, TP1046, TP1047, TP1048, TP1049, TP1050, TP1051, TP1052, TP1053, TP1054, TP1055, TP1056, TP1057, TP1058, TP1059, TP1060, TP1061, TP1062, TP1063, TP1064, TP1065, TP1066, TP1067, TP1068, TP1069, TP1070, TP1071, TP1072, TP1073, TP1074, TP1075, TP1076, TP1077, TP1078, TP1079, TP1080, TP1081, TP1082, TP1083, TP1084, TP1085, TP1086, TP1089, TP1090, TP1091, TP1092, TP1093, TP16, TP2, TP20, TP21, TP22, TP23, TP24, TP25, TP26, TP27, TP28, TP29, TP30, TP31, TP32, TP33, TP34, TP35, TP355, TP357, TP359, TP36, TP37, TP38, TP39, TP40, TP41, TP42, TP43, TP44, TP45, TP46, TP47, TP48, TP49, TP5, TP50, TP51, TP52, TP53, TP54, TP545, TP546, TP55, TP56, TP563, TP564, TP565, TP566, TP567, TP568, TP569, TP57, TP570, TP571, TP572, TP573, TP574, TP575, TP576, TP577, TP578, TP579, TP58, TP580, TP581, TP582, TP583, TP584, TP585, TP586, TP587, TP588, TP589, TP59, TP590, TP591, TP592, TP593, TP594, TP595, TP596, TP597, TP598, TP599, TP60, TP600, TP601, TP602, TP603, TP604, TP605, TP606, TP607, TP608, TP609, TP61, TP610, TP611, TP612, TP62, TP63, TP64, TP640, TP649, TP65, TP650, TP651, TP66, TP660, TP662, TP663, TP664, TP665, TP666, TP667, TP668, TP669, TP67, TP670, TP671, TP672, TP673, TP674, TP675, TP676, TP677, TP678, TP679, TP68, TP680, TP681, TP682, TP683, TP684, TP685, TP686, TP687, TP688, TP689, TP69, TP690, TP691, TP692, TP693, TP694, TP695, TP696, TP697, TP698, TP699, TP70, TP700, TP701, TP702, TP703, TP704, TP705, TP706, TP707, TP708, TP709, TP71, TP710, TP711, TP712, TP713, TP714, TP715, TP716, TP717, TP718, TP719, TP72, TP720, TP721, TP722, TP723, TP724, TP725, TP726, TP727, TP728, TP729, TP73, TP730, TP731, TP732, TP733, TP734, TP735, TP736, TP737, TP738, TP739, TP74, TP740, TP741, TP742, TP743, TP744, TP745, TP746, TP747, TP748, TP749, TP75, TP750, TP751, TP752, TP753, TP754, TP755, TP756, TP757, TP758, TP759, TP76, TP760, TP761, TP762, TP763, TP764, TP765, TP766, TP767, TP768, TP769, TP77, TP770, TP771, TP772, TP773, TP774, TP775, TP776, TP777, TP778, TP779, TP780, TP781, TP782, TP783, TP805, TP806, TP807, TP808, TP809, TP810, TP811, TP812, TP813, TP814, TP815, TP829, TP837, TP844, TP854, TP855, TP873, TP875, TP878, TP879, TP897, TP898, TP905, TP956, TP959, TP960, TP961, TP962, TP963, TP964, TP965, TP966, TP967, TP968, TP969, TP970, TP971, TP972, TP973, TP974, TP975, TP976, TP977, TP978, TP979, TP980, TP981, TP982, TP983, TP984, TP985, TP986, TP987, TP988, TP989, TP990, TP992, TP994, TP999: ~, fp:TestPoint, symbol 16717a:TestPoint_Small
Connections:
- net +1.5V: now also TP1086.1, TP650.1, TP651.1
- net +12V: now also TP736.1, TP813.1, TP815.1
- net +3.3V: now also TP1055.1, TP2.1, TP640.1, TP66.1, TP74.1
- net +3.3VP: now also TP33.1
- net +5V: now also TP1021.1, TP1045.1, TP1053.1, TP1056.1, TP1091.1, TP41.1, TP546.1, TP779.1, TP956.1, TP984.1
- net -12V: now also TP737.1, TP814.1, TP989.1
- net -3.3V: now also TP1084.1, TP1085.1, TP982.1, TP987.1
- net -5.2V: now also TP1092.1, TP1093.1, TP829.1, TP837.1, TP844.1, TP873.1, TP986.1
- net BA_{0}: now also TP612.1
- net BA_{10}: now also TP602.1
- net BA_{11}: now also TP601.1
- net BA_{12}: now also TP600.1
- net BA_{13}: now also TP599.1
- net BA_{14}: now also TP598.1
- net BA_{15}: now also TP597.1
- net BA_{16}: now also TP596.1
- net BA_{17}: now also TP595.1
- net BA_{18}: now also TP594.1
- net BA_{19}: now also TP593.1
- net BA_{1}: now also TP611.1
- net BA_{20}: now also TP592.1
- net BA_{21}: now also TP591.1
- net BA_{22}: now also TP590.1
- net BA_{23}: now also TP589.1
- net BA_{2}: now also TP610.1
- net BA_{3}: now also TP609.1
- net BA_{4}: now also TP608.1
- net BA_{5}: now also TP607.1
- net BA_{6}: now also TP606.1
- net BA_{7}: now also TP605.1
- net BA_{8}: now also TP604.1
- net BA_{9}: now also TP603.1
- net BB_{0}: now also TP588.1
- net BB_{10}: now also TP578.1
- net BB_{11}: now also TP577.1
- net BB_{12}: now also TP576.1
- net BB_{13}: now also TP575.1
- net BB_{14}: now also TP574.1
- net BB_{15}: now also TP573.1
- net BB_{16}: now also TP572.1
- net BB_{17}: now also TP571.1
- net BB_{18}: now also TP570.1
- net BB_{19}: now also TP569.1
- net BB_{1}: now also TP587.1
- net BB_{20}: now also TP568.1
- net BB_{21}: now also TP567.1
- net BB_{22}: now also TP566.1
- net BB_{23}: now also TP565.1
- net BB_{2}: now also TP586.1
- net BB_{3}: now also TP585.1
- net BB_{4}: now also TP584.1
- net BB_{5}: now also TP583.1
- net BB_{6}: now also TP582.1
- net BB_{7}: now also TP581.1
- net BB_{8}: now also TP580.1
- net BB_{9}: now also TP579.1
- net BIF15: now also TP735.1
- net BIF17: now also TP734.1
- net BIF19: now also TP733.1
- net BIF21: now also TP732.1
- net BIF25: now also TP731.1
- net BIF27: now also TP730.1
- net BIF29: now also TP729.1
- net BIF31: now also TP728.1
- net BIF35: now also TP727.1
- net BIF37: now also TP726.1
- net BIF39: now also TP725.1
- net BIF45: now also TP723.1
- net BIF_CLK: now also TP722.1
- net CTRL0L: now also TP747.1
- net CTRL0R: now also TP743.1
- net CTRL10L: now also TP756.1
- net CTRL10R: now also TP757.1
- net CTRL1L: now also TP748.1
- net CTRL1R: now also TP744.1
- net CTRL2L: now also TP749.1
- net CTRL2R: now also TP745.1
- net CTRL3L: now also TP750.1
- net CTRL3R: now also TP746.1
- net CTRL4: now also TP740.1
- net CTRL5WL: now also TP1046.1
- net CTRL5WR: now also TP1047.1
- net CTRL6L: now also TP752.1
- net CTRL6R: now also TP755.1
- net CTRL7L: now also TP754.1
- net CTRL7R: now also TP753.1
- net CTRL9L: now also TP758.1
- net CTRL9R: now also TP759.1
- net EVENT_OUT_{0}: now also TP701.1
- net EVENT_OUT_{1}: now also TP702.1
- net EVENT_OUT_{2}: now also TP703.1
- net EVENT_OUT_{3}: now also TP704.1
- net EVENT_OUT_{4}: now also TP705.1
- net EVENT_OUT_{5}: now also TP706.1
- net EVENT_OUT_{6}: now also TP707.1
- net EVENT_OUT_{7}: now also TP708.1
- net GND: now also C1119.2, C1120.2, TP1018.1, TP1020.1, TP1057.1, TP1068.1, TP34.1, TP35.1, TP355.1, TP40.1, TP545.1, TP649.1, TP715.1, TP73.1, TP739.1, TP77.1, TP776.1, TP777.1, TP778.1, TP780.1, TP781.1, TP782.1, TP783.1, TP878.1, TP960.1, TP981.1; no longer U15.9 (~{HF_{IN}})
- net I2C_A_{0}: now also TP1015.1
- net I2C_CLK: now also TP1012.1
- net IMIO_{0}: now also TP68.1
- net IMIO_{1}: now also TP69.1
- net MASTER_SENSE: now also TP70.1
- net MA_{3}: now also TP1079.1
- net MA_{4}: now also TP1080.1
- net MA_{7}: now also TP1081.1
- net MA_{8}: now also TP1082.1
- net MD_{10}: now also TP1001.1
- net MD_{11}: now also TP1002.1
- net MD_{12}: now also TP1003.1
- net MD_{13}: now also TP1004.1
- net MD_{14}: now also TP1005.1
- net MD_{15}: now also TP1006.1
- net MD_{3}: now also TP20.1
- net MD_{8}: now also TP999.1
- net MD_{9}: now also TP1000.1
- net PC1PR: now also TP854.1
- net PC2PR: now also TP855.1
- net Pod 1/ZOUT_{CLK}: now also TP357.1
- net Pod 1/~{ZOUT_{CLK}}: now also TP359.1
- net SCL: now also TP1017.1
- net SDA: now also TP1016.1
- net STACK_BIAS: now also TP1.1
- net STACK_BIAS_EN: now also TP898.1
- net SYS_CLK: now also TP710.1
- net SYS_CLK_{LEFT}: now also TP711.1
- net SYS_CLK_{RIGHT}: now also TP712.1
- net TEST_CLK_DIV: now also TP1070.1
- net TEST_CLK_{L0}: now also TP53.1
- net TEST_CLK_{L1}: now also TP50.1
- net TEST_CLK_{L2}: now also TP49.1
- net TEST_CLK_{L3}: now also TP46.1
- net TEST_CLK_{L4}: now also TP45.1
- net TEST_CLK_{L}: now also TP54.1
- net TEST_CLK_{R0}: now also TP52.1
- net TEST_CLK_{R1}: now also TP51.1
- net TEST_CLK_{R2}: now also TP48.1
- net TEST_CLK_{R3}: now also TP47.1
- net TEST_CLK_{R4}: now also TP44.1
- net TEST_CLK_{R}: now also TP55.1
- net VREF_{0}: now also TP805.1
- net VREF_{1}: now also TP806.1
- net VREF_{2}: now also TP807.1
- net VREF_{3}: now also TP808.1
- net VREF_{4}: now also TP809.1
- net VREF_{5}: now also TP810.1
- net VREF_{6}: now also TP811.1
- net VREF_{7}: now also TP812.1
- net V_{ZOOM}: now also TP39.1
- net ZCCTRL0: now also TP1073.1
- net ZCCTRL1: now also TP1074.1
- net ZCCTRL2: now also TP1075.1
- net ZCCTRL3: now also TP1076.1
- net ZCCTRL5: now also TP1077.1
- net ZCCTRL6: now also TP1078.1
- net ZOOM_CLK+: now also TP75.1
- net ZOOM_CLK-: now also TP76.1
- net ZOOM_CLK_{EXT+1}+: now also TP59.1
- net ZOOM_CLK_{EXT+1}-: now also TP58.1
- net ZOOM_CLK_{EXT+2}+: now also TP57.1
- net ZOOM_CLK_{EXT+2}-: now also TP56.1
- net ZOOM_CLK_{EXT-1}+: now also TP63.1
- net ZOOM_CLK_{EXT-1}-: now also TP62.1
- net ZOOM_CLK_{EXT-2}+: now also TP65.1
- net ZOOM_CLK_{EXT-2}-: now also TP64.1
- net ZOOM_CLK_{MASTER}+: now also TP61.1
- net ZOOM_CLK_{MASTER}-: now also TP60.1
- net ZOOM_COMPARATOR: now also TP21.1
- net ZOOM_PLL_CTRL: now also TP875.1
- net ~{BIFE_{1}}: now also TP724.1
- net ~{BIFE_{2}}: now also TP1049.1
- net ~{BIFE_{4}}: now also TP1050.1
- net ~{BIFE_{6}}: now also TP1051.1
- net ~{DAC_WR}: now also TP1048.1
- net ~{EN_{TEST}}: now also TP990.1
- net ~{EVENT_LEFT_{0}}: now also TP760.1
- net ~{EVENT_LEFT_{1}}: now also TP761.1
- net ~{EVENT_LEFT_{2}}: now also TP762.1
- net ~{EVENT_LEFT_{3}}: now also TP763.1
- net ~{EVENT_LEFT_{4}}: now also TP764.1
- net ~{EVENT_LEFT_{5}}: now also TP765.1
- net ~{EVENT_LEFT_{6}}: now also TP766.1
- net ~{EVENT_LEFT_{7}}: now also TP767.1
- net ~{EVENT_RIGHT_{0}}: now also TP768.1
- net ~{EVENT_RIGHT_{1}}: now also TP769.1
- net ~{EVENT_RIGHT_{2}}: now also TP770.1
- net ~{EVENT_RIGHT_{3}}: now also TP771.1
- net ~{EVENT_RIGHT_{4}}: now also TP772.1
- net ~{EVENT_RIGHT_{5}}: now also TP773.1
- net ~{EVENT_RIGHT_{6}}: now also TP774.1
- net ~{EVENT_RIGHT_{7}}: now also TP775.1
- net ~{I2C_CS}: now also TP1014.1
- net ~{I2C_EN_{LEFT}}: now also TP1009.1
- net ~{I2C_EN_{RIGHT}}: now also TP1008.1
- net ~{I2C_RD}: now also TP1013.1
- net ~{I2C_RESET}: now also TP1011.1
- net ~{I2C_WR}: now also TP1010.1
- net ~{MEM_CAS_{L0}}: now also TP679.1
- net ~{MEM_CAS_{L10}}: now also TP674.1
- net ~{MEM_CAS_{L11}}: now also TP676.1
- net ~{MEM_CAS_{L12}}: now also TP683.1
- net ~{MEM_CAS_{L13}}: now also TP978.1
- net ~{MEM_CAS_{L14}}: now also TP675.1
- net ~{MEM_CAS_{L15}}: now also TP677.1
- net ~{MEM_CAS_{L16}}: now also TP979.1
- net ~{MEM_CAS_{L1}}: now also TP681.1
- net ~{MEM_CAS_{L2}}: now also TP671.1
- net ~{MEM_CAS_{L3}}: now also TP673.1
- net ~{MEM_CAS_{L4}}: now also TP678.1
- net ~{MEM_CAS_{L5}}: now also TP680.1
- net ~{MEM_CAS_{L6}}: now also TP670.1
- net ~{MEM_CAS_{L7}}: now also TP672.1
- net ~{MEM_CAS_{L8}}: now also TP682.1
- net ~{MEM_CAS_{L9}}: now also TP684.1
- net ~{MEM_CAS_{R0}}: now also TP662.1
- net ~{MEM_CAS_{R10}}: now also TP26.1
- net ~{MEM_CAS_{R11}}: now also TP28.1
- net ~{MEM_CAS_{R12}}: now also TP666.1
- net ~{MEM_CAS_{R13}}: now also TP668.1
- net ~{MEM_CAS_{R14}}: now also TP27.1
- net ~{MEM_CAS_{R15}}: now also TP29.1
- net ~{MEM_CAS_{R16}}: now also TP669.1
- net ~{MEM_CAS_{R1}}: now also TP664.1
- net ~{MEM_CAS_{R2}}: now also TP23.1
- net ~{MEM_CAS_{R3}}: now also TP25.1
- net ~{MEM_CAS_{R4}}: now also TP660.1
- net ~{MEM_CAS_{R5}}: now also TP663.1
- net ~{MEM_CAS_{R6}}: now also TP22.1
- net ~{MEM_CAS_{R7}}: now also TP24.1
- net ~{MEM_CAS_{R8}}: now also TP665.1
- net ~{MEM_CAS_{R9}}: now also TP667.1
- net ~{MEM_RAS_{LL}}: now also TP992.1
- net ~{MEM_RAS_{RL}}: now also TP994.1
- net ~{MEM_SE}: now also TP905.1
- net ~{PROBE_PWR_EN}: now also TP879.1
- net ~{SYS_CLK_{LEFT}}: now also TP713.1
- net ~{SYS_CLK_{RIGHT}}: now also TP714.1
- net ~{SYS_CLK}: now also TP709.1
- net ~{TEST_CLK_EN}: now also TP1071.1
- net at J3.19 (Pin_19), R1291.2, U1.2: now also TP72.1
- net at C1124.1, R1119.1, R213.11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: now also TP716.1
- net at R1052.2, U13.16 (SCLK), U74.1 (CLK/2): now also TP42.1
- net at R1039.1, U74.2 (~{CLK/2}): now also TP43.1
- net at R1046.2, U13.14 (~{CLK}), U74.4 (CLK/4): now also TP1089.1
- net at R1045.2, U13.15 (CLK), U74.5 (~{CLK/4}): now also TP1090.1
- net at R1134.2, R1137.1, U64.36 (TEST_CLK_DIV): now also TP1066.1
- net at RP4.10, U64.118 (~{ZCS_{4}}): now also TP1044.1
- net at RP4.11, U64.117 (~{ZCS_{3}}): now also TP1043.1
- net at RP4.12, U64.116 (~{ZCS_{2}}): now also TP1042.1
- net at RP4.13, U64.115 (~{ZCS_{1}}): now also TP1041.1
- net at RP4.14, U64.114 (~{ZCS_{0}}): now also TP1040.1
- net at RP4.15, U64.102 (~{MEM_CAS_{L16}}): now also TP1039.1
- net at RP4.16, U64.101 (~{MEM_CAS_{L13}}): now also TP1038.1
- net at R1229.1, R1230.1, U16.3 (-): now also TP38.1
- net at R1095.1, U34.29 (~{CLR}): now also TP988.1
- net at C1170.1, R1153.1, U34.3 (V_{REF-}AB)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: now also TP959.1
- net at C1175.2, U34.30 (V_{REF+}GH), U34.39 (V_{REF+}CDEF)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: now also TP961.1
- net at R1116.2, R213.15, U68.1 (Y_{0}): now also TP983.1
- net at R1132.2, R1133.1, U64.35 (~{TEST_CLK_EN}): now also TP1067.1
- net at R1236.1, U15.15 (F_{OUT}), U15.2 (F_{IN}): now also TP31.1
- net at J3.3 (Pin_3), R1290.2, U1.3: now also TP71.1
- net at RP5.9, U64.100 (~{MEM_CAS_{L9}}): now also TP1037.1
- net at RP10.15, RP10.16, U64.135 (CTRL9): now also TP751.1
- net at R1127.1, U64.139 (CTRL8): now also TP742.1
- net at U64.159 (SDI): now also TP1054.1
- net at R1122.1, U64.177 (CTRL4): now also TP741.1
- net at U64.180 (CLK), U66.3 (CLK_{OUT}): now also TP1019.1
- net at U64.207 (DCLK): now also TP1072.1
- net at R1123.1, U64.3 (MODE): now also TP738.1
- net at R1139.2, R1140.2, U64.43 (???): now also TP1065.1
- net at R1141.1, R1147.2, U64.44 (???): now also TP1062.1
- net at R1143.2, R1144.2, U64.48 (???): now also TP1063.1
- net at R1145.2, R1146.2, U64.49 (???): now also TP1064.1
- net at R1103.2, U64.54 (ZOOM_PLL_CTRL/TMS): now also TP1069.1
- net at R1151.2, U64.58 (~{MEM_RAS_{LU}}): now also TP1058.1
- net at R1142.2, U64.59 (~{MEM_RAS_{LL}}): now also TP1059.1
- net at R1149.2, U64.61 (~{MEM_RAS_{RU}}): now also TP1060.1
- net at R1150.1, U64.62 (~{MEM_RAS_{RL}}): now also TP1061.1
- net at RP8.16, U64.65 (~{MEM_CAS_{R6}}): now also TP962.1
- net at RP8.15, U64.66 (~{MEM_CAS_{R2}}): now also TP963.1
- net at RP8.14, U64.67 (~{MEM_CAS_{R7}}): now also TP964.1
- net at RP8.13, U64.68 (~{MEM_CAS_{R3}}): now also TP965.1
- net at RP8.12, U64.69 (~{MEM_CAS_{R10}}): now also TP966.1
- net at RP8.11, U64.70 (~{MEM_CAS_{R14}}): now also TP967.1
- net at RP8.10, U64.71 (~{MEM_CAS_{R11}}): now also TP968.1
- net at RP8.9, U64.72 (~{MEM_CAS_{R15}}): now also TP969.1
- net at RP7.16, U64.73 (~{MEM_CAS_{R4}}): now also TP970.1
- net at RP7.15, U64.74 (~{MEM_CAS_{R0}}): now also TP971.1
- net at RP7.14, U64.75 (~{MEM_CAS_{R5}}): now also TP972.1
- net at RP7.13, U64.76 (~{MEM_CAS_{R1}}): now also TP973.1
- net at RP7.12, U64.77 (~{MEM_CAS_{R8}}): now also TP974.1
- net at RP7.11, U64.81 (~{MEM_CAS_{R12}}): now also TP975.1
- net at RP7.10, U64.82 (~{MEM_CAS_{R9}}): now also TP976.1
- net at RP7.9, U64.83 (~{MEM_CAS_{R13}}): now also TP977.1
- net at RP6.16, U64.84 (~{MEM_CAS_{R16}}): now also TP1022.1
- net at RP6.15, U64.85 (~{MEM_CAS_{L6}}): now also TP1023.1
- net at RP6.14, U64.86 (~{MEM_CAS_{L2}}): now also TP1024.1
- net at RP6.13, U64.87 (~{MEM_CAS_{L7}}): now also TP1025.1
- net at RP6.12, U64.88 (~{MEM_CAS_{L3}}): now also TP1026.1
- net at RP6.11, U64.89 (~{MEM_CAS_{L10}}): now also TP1027.1
- net at RP6.10, U64.90 (~{MEM_CAS_{L14}}): now also TP1028.1
- net at RP6.9, U64.91 (~{MEM_CAS_{L11}}): now also TP1029.1
- net at RP5.16, U64.92 (~{MEM_CAS_{L15}}): now also TP1030.1
- net at RP5.15, U64.93 (~{MEM_CAS_{L4}}): now also TP1031.1
- net at RP5.14, U64.94 (~{MEM_CAS_{L0}}): now also TP1032.1
- net at RP5.13, U64.95 (~{MEM_CAS_{L5}}): now also TP1033.1
- net at RP5.12, U64.96 (~{MEM_CAS_{L1}}): now also TP1034.1
- net at RP5.11, U64.97 (~{MEM_CAS_{L8}}): now also TP1035.1
- net at RP5.10, U64.99 (~{MEM_CAS_{L12}}): now also TP1036.1
- net at C1109.1, R1106.1, R1107.1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: now also TP985.1
- net at C1235.1, R1233.1, R1240.1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: now also TP30.1
- net at C1240.1, R1044.1, R1233.2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: now also TP16.1
- net at Q1.1 (B), R1093.1: now also TP897.1
- net at C1241.1, R1038.1, R1240.2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: now also TP5.1
- net at RP16.1, RP9.16, U76.18 (Y0): now also TP685.1
- net at RP16.2, RP9.15, U76.17 (Y1): now also TP686.1
- net at RP16.3, RP9.14, U76.16 (Y2): now also TP687.1
- net at RP16.4, RP9.13, U76.15 (Y3): now also TP688.1
- net at RP16.5, RP9.12, U76.14 (Y4): now also TP689.1
- net at RP16.6, RP9.11, U76.13 (Y5): now also TP690.1
- net at RP16.7, RP9.10, U76.12 (Y6): now also TP691.1
- net at RP16.8, RP9.9, U76.11 (Y7): now also TP692.1
- net at R1115.2, R213.13, U68.2 (~{Y_{0}}): now also TP1052.1
- net at R1166.1, RP13.16: now also TP564.1
- net at R1165.1, RP12.1: now also TP563.1
- net at C1123.1, R1113.2, U68.4 (~{Y_{1}}): now also TP719.1
- net at C1123.2, R1118.1, R213.10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: now also TP717.1
- net at C1332.1, J6.16 (Pin_16), R1249.1: now also TP67.1
- net at R1111.2, U68.6 (~{A}): now also TP720.1
- net at R1043.2, U15.14 (~{F_{OUT}}), U15.3 (~{F_{IN}}): now also TP32.1
- net at R1237.2, U15.18 (~{R_{IN}}), U73.6: now also TP37.1
- net at R1239.2, U15.19 (R_{IN}), U73.7: now also TP36.1
- net at C1124.2, R1114.2, U68.3 (Y_{1}): now also TP718.1
- net at U67.10 (AO_{5}), U76.6 (A4): now also TP697.1
- net at U67.12 (AO_{6}), U76.7 (A5): now also TP698.1
- net at U67.16 (AO_{7}), U76.8 (A6): now also TP699.1
- net at U67.20 (AO_{8}), U76.9 (A7): now also TP700.1
- net at U67.4 (AO_{3}), U76.4 (A2): now also TP695.1
- net at U67.50 (AO_{1}), U76.2 (A0): now also TP693.1
- net at U67.52 (AO_{2}), U76.3 (A1): now also TP694.1
- net at U67.6 (AO_{4}), U76.5 (A3): now also TP696.1
- net at R1112.2, U68.7 (A): now also TP721.1
- net at R1120.2, U66.1 (OE/~{ST}): now also TP1083.1
- net at C1111.1, R1108.1, R1109.1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: now also TP980.1
- no-connect marks 41 -> 40
Other:
- moved on the sheet: R1093, R1103, R1111, R1112, R1122, R1127, R1142, R1149, R1150, R1151
