File: original/pod_cmp.kicad_sch (KiCad schematic)
At the start: 104 parts, among them U69 1NB4-5036, U70 1NB4-5036

Commit message: clean up routing & add test points on original design
Parts:
- added TP507, TP509, TP511, TP513, TP515, TP517, TP519, TP521, TP527, TP529, TP531, TP535, TP537, TP539, TP541, TP543, TP550, TP552, TP785, TP787, TP789, TP791, TP793, TP795, TP797, TP799, TP801, TP803, TP81, TP83, TP838, TP845, TP847, TP85, TP87: ~, fp:TestPoint, symbol 16717a:TestPoint_Small
Connections:
- net +3.3V: now also TP552.1, TP845.1, TP847.1
- net -3.3V: now also TP838.1
- net GND: now also TP550.1
- net V_{BB}_{H}: now also TP83.1
- net V_{BB}_{L}: now also TP81.1
- net ZOUT_{0}: now also TP543.1
- net ZOUT_{10}: now also TP517.1
- net ZOUT_{11}: now also TP515.1
- net ZOUT_{12}: now also TP513.1
- net ZOUT_{13}: now also TP511.1
- net ZOUT_{14}: now also TP509.1
- net ZOUT_{15}: now also TP507.1
- net ZOUT_{1}: now also TP541.1
- net ZOUT_{2}: now also TP539.1
- net ZOUT_{3}: now also TP537.1
- net ZOUT_{5}: now also TP531.1
- net ZOUT_{6}: now also TP529.1
- net ZOUT_{7}: now also TP527.1
- net ZOUT_{8}: now also TP521.1
- net ZOUT_{9}: now also TP519.1
- net ZV_{BB}_{L}: now also TP535.1
- net at R328.1, U69.19 (V_{BB}): now also TP789.1
- net at R328.5, U69.25 (OUT_{1}): now also TP785.1
- net at R328.3, U69.27 (OUT_{0}): now also TP787.1
- net at R329.5, U69.7 (OUT_{8}): now also TP793.1
- net at R329.3, U69.8 (~{OUT_{8}}): now also TP791.1
- net at R335.7, U70.10 (OUT_{7}): now also TP801.1
- net at R335.5, U70.12 (OUT_{6}): now also TP803.1
- net at R334.3, U70.23 (OUT_{2}): now also TP799.1
- net at R334.1, U70.25 (OUT_{1}): now also TP797.1
- net at R329.7, U70.27 (OUT_{0}): now also TP795.1
- net at R1267.1, R328.16: now also TP87.1
- net at R1269.1, R334.10: now also TP85.1
