File: original/pod_cmp_top.kicad_sch (KiCad schematic)
At the start: 104 parts, among them U3 1NB4-5036, U4 1NB4-5036

Commit message: clean up routing & add test points on original design
Parts:
- added TP831, TP842, TP850, TP852, TP865, TP89, TP91, TP93, TP95: ~, fp:TestPoint, symbol 16717a:TestPoint_Small
Connections:
- net -3.3V: now also TP865.1
- net -5.2V: now also TP852.1
- net GND: now also TP850.1
- net V_{BB}_{H}: now also TP93.1
- net V_{BB}_{L}: now also TP89.1
- net at R1018.1, R126.14: now also TP95.1
- net at R126.3, U3.19 (V_{BB}): now also TP831.1
- net at R131.1, U4.19 (V_{BB}): now also TP842.1
- net at R1020.1, R131.16: now also TP91.1
