File: original/ram.kicad_sch (KiCad schematic)
At the start: 74 parts, among them U25 MSM5416283, U26 MSM5416283, U27 MSM5416283, U28 MSM5416283, U29 MSM5416283, U30 MSM5416283, U31 MSM5416283, U32 MSM5416283, U33 MSM5416283, U35 MSM5416283, U36 MSM5416283, U37 MSM5416283, U38 MSM5416283, U39 MSM5416283, U40 MSM5416283, U41 MSM5416283, U42 MSM5416283, U43 MSM5416283, U46 MSM5416283, U47 MSM5416283, U48 MSM5416283, U49 MSM5416283, U50 MSM5416283, U51 MSM5416283, U52 MSM5416283, U53 MSM5416283, U54 MSM5416283, U55 MSM5416283, U56 MSM5416283, U57 MSM5416283, U58 MSM5416283, U59 MSM5416283, U60 MSM5416283, U61 MSM5416283

Commit message: clean up routing & add test points on original design
Parts:
- added TP10, TP1007, TP11, TP12, TP13, TP14, TP15, TP17, TP18, TP19, TP3, TP354, TP4, TP6, TP7, TP8, TP899, TP9, TP900, TP901, TP902, TP903, TP904, TP906, TP907, TP908, TP909, TP910, TP911, TP912, TP913, TP914, TP915, TP916, TP917, TP918, TP919, TP920, TP921, TP922, TP923, TP924, TP925, TP926, TP927, TP928, TP929, TP930, TP931, TP932, TP933, TP934, TP935, TP936, TP937, TP938, TP939, TP940, TP941, TP942, TP943, TP944, TP945, TP946, TP947, TP948, TP949, TP950, TP951, TP952, TP953, TP954, TP955, TP957, TP958: ~, fp:TestPoint, symbol 16717a:TestPoint_Small
Connections:
- net +5V: now also TP12.1, TP13.1, TP3.1, TP6.1, TP9.1, TP903.1, TP906.1, TP907.1, TP909.1, TP912.1, TP915.1, TP917.1, TP919.1, TP922.1, TP923.1, TP925.1, TP928.1, TP931.1, TP933.1, TP935.1, TP938.1, TP942.1, TP944.1, TP946.1, TP948.1, TP949.1, TP951.1, TP954.1, TP958.1
- net GND: now also TP10.1, TP1007.1, TP11.1, TP14.1, TP4.1, TP7.1, TP8.1, TP904.1, TP908.1, TP910.1, TP911.1, TP913.1, TP914.1, TP916.1, TP918.1, TP920.1, TP921.1, TP924.1, TP926.1, TP927.1, TP929.1, TP930.1, TP932.1, TP934.1, TP936.1, TP937.1, TP939.1, TP940.1, TP941.1, TP943.1, TP945.1, TP947.1, TP950.1, TP952.1, TP953.1, TP955.1, TP957.1
- net MA_{2}: now also TP15.1
- net SDR_{129}: now also TP17.1
- net SDR_{130}: now also TP18.1
- net SDR_{132}: now also TP19.1
- net SDR_{134}: now also TP354.1
- net SDR_{25}: now also TP902.1
- net SDR_{27}: now also TP901.1
- net SDR_{29}: now also TP900.1
- net SDR_{31}: now also TP899.1
